File: kicad/inversor.kicad_sch (KiCad schematic)
At the start: 64 parts, among them J1 VCC, J2 PWM, J3 LCD 16x2, J4 MainFan, J5 380VFreed, J6 PRO_MINI_L, J7 PRO_MINI_T, J8 PRO_MINI_R, Q1 SSF6014D, Q2 TIP120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

Commit message: FIX: VCC Arduino 5v en lugar de VCC FIX: Divisor de tension para sensor de voltaje de batería con resistencia en la parte de vcc en lugar de gnd
Connections:
- net +5V: now also J8.9 (Pin_9)
- net GND: now also RV4.3; no longer R15.2
- net VCC: now also R15.1; no longer J8.9 (Pin_9), RV4.1
- new net: R15.2, RV4.1
Other:
- moved on the sheet: R15, RV4

Commit message: Fix: - Agregado condensador en la linea VCC - Agregada línea entre D13 del arduino y DS del SG3525 para poder detenerlo - Ajustes en pistas
Parts:
- added C14: 250nF, Capacitor_THT:CP_Radial_D5.0mm_P2.50mm, symbol Device:C_Polarized
- R22: footprint Resistor_THT:R_Axial_DIN0207_L6.3mm_D2.5mm_P10.16mm_Horizontal -> Resistor_THT:R_Axial_DIN0207_L6.3mm_D2.5mm_P7.62mm_Horizontal
Connections:
- net SD is gone; now on net D13: J2.2 (Pin_2), U3.10 (SD)
- net GND: now also C14.2
- net VCC: now also C14.1
Changed lines of the file:
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@@
   (junction (at 133.35 63.5) (diameter 0) (color 0 0 0 0)
   )
+  (junction (at 29.21 29.21) (diameter 0) (color 0 0 0 0)
+  )
   (junction (at 135.89 21.59) (diameter 0) (color 0 0 0 0)
   )
@@
   (junction (at 207.01 97.79) (diameter 0) (color 0 0 0 0)
   )
+  (junction (at 26.67 140.97) (diameter 0) (color 0 0 0 0)
+  )
   (junction (at 132.08 161.29) (diameter 0) (color 0 0 0 0)
   )
@@
     (stroke (width 0) (type default) (color 0 0 0 0))
   )
+  (wire (pts (xy 29.21 29.21) (xy 29.21 33.02))
+    (stroke (width 0) (type default) (color 0 0 0 0))
+  )
   (wire (pts (xy 26.67 21.59) (xy 30.48 21.59))
     (stroke (width 0) (type default) (color 0 0 0 0))
   )
+  (wire (pts (xy 26.67 142.24) (xy 26.67 140.97))
+    (stroke (width 0) (type default) (color 0 0 0 0))
+  )
   (wire (pts (xy 43.18 95.25) (xy 54.61 95.25))
     (stroke (width 0) (type default) (color 0 0 0 0))
@@
     (stroke (width 0) (type default) (color 0 0 0 0))
   )
+  (wire (pts (xy 29.21 29.21) (xy 26.67 29.21))
+    (stroke (width 0) (type default) (color 0 0 0 0))
+  )
   (wire (pts (xy 158.75 90.17) (xy 158.75 83.82))
     (stroke (width 0) (type default) (color 0 0 0 0))
@@
     (stroke (width 0) (type default) (color 0 0 0 0))
   )
+  (wire (pts (xy 26.67 140.97) (xy 30.48 140.97))
+    (stroke (width 0) (type default) (color 0 0 0 0))
+  )
   (wire (pts (xy 201.93 20.32) (xy 213.36 20.32))
     (stroke (width 0) (type default) (color 0 0 0 0))
@@
     (stroke (width 0) (type default) (color 0 0 0 0))
   )
+  (wire (pts (xy 30.48 33.02) (xy 29.21 33.02))
+    (stroke (width 0) (type default) (color 0 0 0 0))
+  )
   (wire (pts (xy 132.08 138.43) (xy 166.37 138.43))
     (stroke (width 0) (type default) (color 0 0 0 0))
@@
     (stroke (width 0) (type default) (color 0 0 0 0))
   )
+  (wire (pts (xy 26.67 149.86) (xy 26.67 151.13))
+    (stroke (width 0) (type default) (color 0 0 0 0))
+  )
   (wire (pts (xy 53.34 107.95) (xy 53.34 115.57))
     (stroke (width 0) (type default) (color 0 0 0 0))
@@
     (stroke (width 0) (type default) (color 0 0 0 0))
   )
-  (wire (pts (xy 29.21 29.21) (xy 26.67 29.21))
+  (wire (pts (xy 30.48 29.21) (xy 29.21 29.21))
     (stroke (width 0) (type default) (color 0 0 0 0))
   )
@@
     (stroke (width 0) (type default) (color 0 0 0 0))
   )
-  (wire (pts (xy 22.86 140.97) (xy 30.48 140.97))
+  (wire (pts (xy 26.67 151.13) (xy 38.1 151.13))
+    (stroke (width 0) (type default) (color 0 0 0 0))
+  )
+  (wire (pts (xy 22.86 140.97) (xy 26.67 140.97))
     (stroke (width 0) (type default) (color 0 0 0 0))
   )
@@
     (stroke (width 0) (type default) (color 0 0 0 0))
   )
-  (wire (pts (xy 26.67 31.75) (xy 30.48 31.75))
+  (wire (pts (xy 26.67 31.75) (xy 26.67 36.83))
     (stroke (width 0) (type default) (color 0 0 0 0))
   )
@@
     )
   )
+  (global_label "D13" (shape input) (at 30.48 33.02 0) (fields_autoplaced)
+    (effects (font (size 1.27 1.27)) (justify left))
+    (property "Referencias entre hojas" "${INTERSHEET_REFS}" (id 0) (at 36.5821 32.9406 0)
+      (effects (font (size 1.27 1.27)) (justify left) hide)
+    )
+  )
   (global_label "D9" (shape input) (at 246.38 149.86 180) (fields_autoplaced)
     (effects (font (size 1.27 1.27)) (justify right))
@@
     )
   )
-  (global_label "SD" (shape input) (at 29.21 29.21 0) (fields_autoplaced)
+  (global_label "SD" (shape input) (at 30.48 29.21 0) (fields_autoplaced)
     (effects (font (size 1.27 1.27)) (justify left))
-    (property "Referencias entre hojas" "${INTERSHEET_REFS}" (id 0) (at 34.1026 29.2894 0)
+    (property "Referencias entre hojas" "${INTERSHEET_REFS}" (id 0) (at 35.3726 29.2894 0)
       (effects (font (size 1.27 1.27)) (justify left) hide)
     )
@@
     (property "Reference" "R22" (id 0) (at 223.52 22.86 90))
     (property "Value" "10K" (id 1) (at 223.52 17.78 90))
-    (property "Footprint" "Resistor_THT:R_Axial_DIN0207_L6.3mm_D2.5mm_P10.16mm_Horizontal" (id 2) (at 223.52 22.098 90)
+    (property "Footprint" "Resistor_THT:R_Axial_DIN0207_L6.3mm_D2.5mm_P7.62mm_Horizontal" (id 2) (at 223.52 22.098 90)
       (effects (font (size 1.27 1.27)) hide)
     )
@@
     (pin "2")
   )
-  (symbol (lib_id "power:+15V") (at 30.48 31.75 270) (unit 1)
+  (symbol (lib_id "power:+15V") (at 26.67 36.83 270) (unit 1)
     (in_bom yes) (on_board yes) (fields_autoplaced)
-    (property "Reference" "#PWR04" (id 0) (at 26.67 31.75 0)
+    (property "Reference" "#PWR04" (id 0) (at 22.86 36.83 0)
       (effects (font (size 1.27 1.27)) hide)
     )
-    (property "Value" "+15V" (id 1) (at 34.29 31.7499 90)
+    (property "Value" "+15V" (id 1) (at 30.48 36.8299 90)
       (effects (font (size 1.27 1.27)) (justify left))
     )
-    (property "Footprint" "" (id 2) (at 30.48 31.75 0)
+    (property "Footprint" "" (id 2) (at 26.67 36.83 0)
       (effects (font (size 1.27 1.27)) hide)
     )
-    (property "Datasheet" "" (id 3) (at 30.48 31.75 0)
+    (property "Datasheet" "" (id 3) (at 26.67 36.83 0)
       (effects (font (size 1.27 1.27)) hide)
     )
@@
     (pin "2")
   )
+  (symbol (lib_id "Device:C_Polarized") (at 26.67 146.05 0) (unit 1)
+    (in_bom yes) (on_board yes)
+    (property "Reference" "C14" (id 0) (at 19.05 146.05 0)
+      (effects (font (size 1.27 1.27)) (justify left))
+    )
+    (property "Value" "250nF" (id 1) (at 19.05 148.59 0)
+      (effects (font (size 1.27 1.27)) (justify left))
+    )
+    (property "Footprint" "Capacitor_THT:CP_Radial_D5.0mm_P2.50mm" (id 2) (at 27.6352 149.86 0)
+      (effects (font (size 1.27 1.27)) hide)
+    )
+    (property "Datasheet" "~" (id 3) (at 26.67 146.05 0)
+      (effects (font (size 1.27 1.27)) hide)
+    )
+    (pin "1")
+    (pin "2")
+  )
   (symbol (lib_id "Device:R") (at 72.39 50.8 0) (unit 1)
     (in_bom yes) (on_board yes) (fields_autoplaced)
@@
       (reference "C13") (unit 1) (value "470uF") (footprint "Capacitor_THT:CP_Radial_D4.0mm_P2.00mm")
     )
+    (path "/ee1b84d0-2880-4387-9006-16f7e093273d"
+      (reference "C14") (unit 1) (value "250nF") (footprint "Capacitor_THT:CP_Radial_D5.0mm_P2.50mm")
+    )
     (path "/fed7b71c-6b44-4677-b167-f2a784fdeee3"
       (reference "D1") (unit 1) (value "D") (footprint "Diode_THT:D_A-405_P7.62mm_Horizontal")
@@
     )
     (path "/83730947-2a66-4670-adfe-0f17d1d7ee9f"
-      (reference "R22") (unit 1) (value "10K") (footprint "Resistor_THT:R_Axial_DIN0207_L6.3mm_D2.5mm_P10.16mm_Horizontal")
+      (reference "R22") (unit 1) (value "10K") (footprint "Resistor_THT:R_Axial_DIN0207_L6.3mm_D2.5mm_P7.62mm_Horizontal")
     )
     (path "/9f0e3837-17f4-4a88-adea-2fbbd4b5a002/0f1f8f32-f06a-45fa-b50e-e942d69f216e"
